Commit message: Add KHI unofficial version to the repo

File: khi_description/srdf/btp/khi_macro.srdf.xacro (robot description, xacro)
@@ -41,4 +41,20 @@
     <disable_collisions link1="${prefix}link4" link2="${prefix}link6" reason="Never" />
     <disable_collisions link1="${prefix}link5" link2="${prefix}link6" reason="Adjacent" />
+    <disable_collisions link1="${prefix}link2" link2="${prefix}parallel_arm2" reason="Adjacent" />
+    <disable_collisions link1="${prefix}parallel_arm1" link2="${prefix}base_link" reason="Never" />
+    <disable_collisions link1="${prefix}parallel_arm1" link2="${prefix}link1" reason="Adjacent" />
+    <disable_collisions link1="${prefix}parallel_arm1" link2="${prefix}link2" reason="Never" />
+    <disable_collisions link1="${prefix}parallel_arm1" link2="${prefix}link3" reason="Never" />
+    <disable_collisions link1="${prefix}parallel_arm1" link2="${prefix}link4" reason="Never" />
+    <disable_collisions link1="${prefix}parallel_arm1" link2="${prefix}link5" reason="Never" />
+    <disable_collisions link1="${prefix}parallel_arm1" link2="${prefix}link6" reason="Never" />
+    <disable_collisions link1="${prefix}parallel_arm1" link2="${prefix}parallel_arm2" reason="Adjacent" />
+    <disable_collisions link1="${prefix}parallel_arm2" link2="${prefix}base_link" reason="Never" />
+    <disable_collisions link1="${prefix}parallel_arm2" link2="${prefix}link1" reason="Never" />
+    <disable_collisions link1="${prefix}parallel_arm2" link2="${prefix}link2" reason="Adjacent" />
+    <disable_collisions link1="${prefix}parallel_arm2" link2="${prefix}link3" reason="Adjacent" />
+    <disable_collisions link1="${prefix}parallel_arm2" link2="${prefix}link4" reason="Never" />
+    <disable_collisions link1="${prefix}parallel_arm2" link2="${prefix}link5" reason="Never" />
+    <disable_collisions link1="${prefix}parallel_arm2" link2="${prefix}link6" reason="Never" />
   </xacro:macro>
 </robot>

File: khi_description/urdf/btp/get_mechanical_parameters.xacro (robot description, xacro)
@@ -1,5 +1,10 @@
 <?xml version="1.0"?>
 <robot xmlns:xacro="http://ros.org/wiki/xacro">
-  <xacro:property name="is_parallel" value="false"/>
+  <xacro:if value="${robot_name == 'bx300l-b001'}">
+    <xacro:property name="is_parallel" value="true"/>
+  </xacro:if>
+  <xacro:unless value="${robot_name == 'bx300l-b001'}">
+    <xacro:property name="is_parallel" value="false"/>
+  </xacro:unless>
   <xacro:property name="mech_para_path" value="$(find khi_description)/config/$(arg robot_series)/$(arg robot_name)/mechanical_parameters.yaml"/>
   <xacro:property name="mechanical_parameters" value="${xacro.load_yaml(mech_para_path)}"/>

File: khi_description/urdf/bx/khi.ros2_control.xacro (robot description, xacro)
@@ -7,5 +7,4 @@
     simulation
     use_gazebo
-    use_gz
     robot_ip
     robot_controller
@@ -20,6 +19,5 @@
     ft_sensor
     ">
-    <xacro:property name="safe_robot_name" value="${robot_name.replace('-', '_')}" />
-    <ros2_control name="${safe_robot_name}" type="system">
+    <ros2_control name="${robot_name}" type="system">
       <xacro:include filename="$(find khi_description)/urdf/$(arg robot_series)/get_mechanical_parameters.xacro"/>
       <xacro:include filename="$(find khi_description)/urdf/$(arg robot_series)/get_joint_limits.xacro"/>
@@ -32,8 +30,5 @@
           <plugin>gazebo_ros2_control/GazeboSystem</plugin>
         </xacro:if>
-        <xacro:if value="${use_gz}">
-          <plugin>gz_ros2_control/GazeboSimSystem</plugin>
-        </xacro:if>
-        <xacro:unless value="${use_gazebo or use_gz}">
+        <xacro:unless value="${use_gazebo}">
           <plugin>khi_hardware/KhiHardwareInterface</plugin>
           <param name="robot_name">$(arg robot_name)</param>
@@ -118,5 +113,5 @@
         <param name="arm">arm1</param>
       </joint>
-      <xacro:if value="${use_gazebo or use_gz}">
+      <xacro:if value="${use_gazebo}">
         <xacro:if value="${is_parallel}">
           <joint name="${prefix}parallel_joint1">

File: khi_description/urdf/bxp/khi.ros2_control.xacro (robot description, xacro)
@@ -20,6 +20,5 @@
     ft_sensor
     ">
-    <xacro:property name="safe_robot_name" value="${robot_name.replace('-', '_')}" />
-    <ros2_control name="${safe_robot_name}" type="system">
+    <ros2_control name="${robot_name}" type="system">
       <xacro:include filename="$(find khi_description)/urdf/$(arg robot_series)/get_mechanical_parameters.xacro"/>
       <xacro:include filename="$(find khi_description)/urdf/$(arg robot_series)/get_joint_limits.xacro"/>

File: khi_description/urdf/khi.urdf.xacro (robot description, xacro)
@@ -21,5 +21,4 @@
   <xacro:include filename="$(find khi_description)/urdf/$(arg robot_series)/khi.ros2_control.xacro"/>
   <xacro:include filename="$(find khi_description)/urdf/khi.gazebo.xacro"/>
-  <xacro:include filename="$(find khi_description)/urdf/khi.gz.xacro"/>
   <!-- instantiate robot -->
   <xacro:khi_joint_link prefix="$(arg prefix)" robot_series="$(arg robot_series)" robot_name="$(arg robot_name)"/>
@@ -46,6 +45,3 @@
     <xacro:khi_gazebo robot_series="$(arg robot_series)" robot_controller="$(arg robot_controller)"/>
   </xacro:if>
-  <xacro:if value="$(arg use_gz)">
-    <xacro:khi_gz robot_series="$(arg robot_series)" robot_controller="$(arg robot_controller)"/>
-  </xacro:if>
 </robot>

File: khi_description/urdf/rs/khi.ros2_control.xacro (robot description, xacro)
@@ -20,6 +20,5 @@
     ft_sensor
     ">
-    <xacro:property name="safe_robot_name" value="${robot_name.replace('-', '_')}" />
-    <ros2_control name="${safe_robot_name}" type="system">
+    <ros2_control name="${robot_name}" type="system">
       <xacro:include filename="$(find khi_description)/urdf/$(arg robot_series)/get_mechanical_parameters.xacro"/>
       <xacro:include filename="$(find khi_description)/urdf/$(arg robot_series)/get_joint_limits.xacro"/>

File: khi_description/urdf/wd/khi.ros2_control.xacro (robot description, xacro)
@@ -20,6 +20,5 @@
     ft_sensor
     ">
-    <xacro:property name="safe_robot_name" value="${robot_name.replace('-', '_')}" />
-    <ros2_control name="${safe_robot_name}" type="system">
+    <ros2_control name="${robot_name}" type="system">
       <xacro:include filename="$(find khi_description)/urdf/$(arg robot_series)/get_mechanical_parameters.xacro"/>
       <xacro:include filename="$(find khi_description)/urdf/$(arg robot_series)/get_joint_limits.xacro"/>
